File: schematic/FPGA_NES_controller.sch (EAGLE design)
At the start: 4 parts, among them IC1 74165N, IC2 74LS04N

Commit message: corrected schematic
Parts:
- added R1, R2: 3.6k, rcl:R-US_V526-0
Connections:
- net CLK: now also R1.1
- net LATCH: now also R2.1
- net VCC: now also R1.2, R2.2
Changed lines of the file:
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@@
 <part name="SUPPLY3" library="supply2" deviceset="GND" device=""/>
 <part name="P+1" library="supply1" deviceset="VCC" device=""/>
+<part name="R1" library="rcl" deviceset="R-US_" device="V526-0" value="3.6k"/>
+<part name="R2" library="rcl" deviceset="R-US_" device="V526-0" value="3.6k"/>
+<part name="P+2" library="supply1" deviceset="VCC" device=""/>
+<part name="P+3" library="supply1" deviceset="VCC" device=""/>
 </parts>
 <sheets>
@@
 <instance part="SUPPLY1" gate="GND" x="-17.78" y="48.26"/>
 <instance part="NES_PORT" gate="A" x="63.5" y="99.06"/>
-<instance part="SUPPLY2" gate="GND" x="91.44" y="99.06"/>
+<instance part="SUPPLY2" gate="GND" x="76.2" y="91.44"/>
 <instance part="SUPPLY3" gate="GND" x="48.26" y="38.1"/>
 <instance part="P+1" gate="VCC" x="48.26" y="106.68"/>
+<instance part="R1" gate="G$1" x="83.82" y="114.3" rot="R90"/>
+<instance part="R2" gate="G$1" x="91.44" y="114.3" rot="R90"/>
+<instance part="P+2" gate="VCC" x="83.82" y="121.92"/>
+<instance part="P+3" gate="VCC" x="91.44" y="121.92"/>
 </instances>
 <busses>
@@
 <pinref part="NES_PORT" gate="A" pin="2"/>
 <pinref part="SUPPLY2" gate="GND" pin="GND"/>
-<wire x1="68.58" y1="104.14" x2="91.44" y2="104.14" width="0.1524" layer="91"/>
-<wire x1="91.44" y1="104.14" x2="91.44" y2="101.6" width="0.1524" layer="91"/>
+<wire x1="68.58" y1="104.14" x2="76.2" y2="104.14" width="0.1524" layer="91"/>
+<wire x1="76.2" y1="104.14" x2="76.2" y2="93.98" width="0.1524" layer="91"/>
 </segment>
 <segment>
@@
 <pinref part="NES_PORT" gate="A" pin="4"/>
 <wire x1="68.58" y1="101.6" x2="83.82" y2="101.6" width="0.1524" layer="91"/>
-<label x="76.2" y="101.6" size="1.778" layer="95"/>
+<label x="93.98" y="101.6" size="1.778" layer="95"/>
+<pinref part="R1" gate="G$1" pin="1"/>
+<wire x1="83.82" y1="101.6" x2="101.6" y2="101.6" width="0.1524" layer="91"/>
+<wire x1="83.82" y1="101.6" x2="83.82" y2="109.22" width="0.1524" layer="91"/>
+<junction x="83.82" y="101.6"/>
 </segment>
 <segment>
@@
 <segment>
 <pinref part="NES_PORT" gate="A" pin="6"/>
-<wire x1="68.58" y1="99.06" x2="83.82" y2="99.06" width="0.1524" layer="91"/>
-<label x="76.2" y="99.06" size="1.778" layer="95"/>
+<wire x1="68.58" y1="99.06" x2="91.44" y2="99.06" width="0.1524" layer="91"/>
+<label x="93.98" y="99.06" size="1.778" layer="95"/>
+<pinref part="R2" gate="G$1" pin="1"/>
+<wire x1="91.44" y1="99.06" x2="101.6" y2="99.06" width="0.1524" layer="91"/>
+<wire x1="91.44" y1="99.06" x2="91.44" y2="109.22" width="0.1524" layer="91"/>
+<junction x="91.44" y="99.06"/>
 </segment>
 <segment>
@@
 <segment>
 <pinref part="NES_PORT" gate="A" pin="8"/>
-<wire x1="68.58" y1="96.52" x2="83.82" y2="96.52" width="0.1524" layer="91"/>
-<label x="76.2" y="96.52" size="1.778" layer="95"/>
+<wire x1="68.58" y1="96.52" x2="101.6" y2="96.52" width="0.1524" layer="91"/>
+<label x="93.98" y="96.52" size="1.778" layer="95"/>
 </segment>
 <segment>
@@
 <wire x1="48.26" y1="101.6" x2="48.26" y2="104.14" width="0.1524" layer="91"/>
 </segment>
+<segment>
+<pinref part="R1" gate="G$1" pin="2"/>
+<pinref part="P+2" gate="VCC" pin="VCC"/>
+</segment>
+<segment>
+<pinref part="R2" gate="G$1" pin="2"/>
+<pinref part="P+3" gate="VCC" pin="VCC"/>
+</segment>
 </net>
